Commit message: instead of using primitive shapes, use directly the meshes for collision checking

File: franka_description/robots/hand.xacro (robot description, xacro)
@@ -17,4 +17,9 @@
       </visual>
       <collision>
+        <geometry>
+          <mesh filename="package://franka_description/meshes/visual/hand.dae"/>
+        </geometry>
+      </collision>
+      <!--collision>
         <origin xyz="0 0 0.04" rpy="0 ${pi/2} ${pi/2}"/>
         <geometry>
@@ -51,5 +56,5 @@
           <sphere radius="${0.02+safety_distance}"  />
         </geometry>
-      </collision>
+      </collision-->
     </link>
     <link name="${ns}_leftfinger">
@@ -59,4 +64,9 @@
         </geometry>
       </visual>
+       <collision>
+        <geometry>
+          <mesh filename="package://franka_description/meshes/visual/finger.dae"/>
+        </geometry>
+      </collision>
     </link>
     <link name="${ns}_rightfinger">
@@ -67,4 +77,10 @@
         </geometry>
       </visual>
+      <collision>
+        <origin xyz="0 0 0" rpy="0 0 ${pi}"/>
+        <geometry>
+          <mesh filename="package://franka_description/meshes/visual/finger.dae"/>
+        </geometry>
+      </collision>
    </link>
     <joint name="${ns}_finger_joint1" type="prismatic">
