Commit message: add table on which the panda is fixed directly in the urdf

File: franka_description/robots/panda_arm.xacro (robot description, xacro)
@@ -11,4 +11,17 @@
       </joint>
     </xacro:unless>
+    <link name="table_link">
+    <visual>
+      <geometry>
+        <box size="1.68 0.83 0.768"/>
+      </geometry>
+      <origin rpy="0.0 0.0 0.0" xyz="0 0 0.384"/>
+    </visual>
+    </link>
+    <joint name="table_to_${arm_id}" type="fixed">
+      <parent link="table_link"/>
+      <child link="${arm_id}_link0"/>
+      <origin xyz="-0.558 0.175 0.768"/>
+    </joint>
     <link name="${arm_id}_link0">
       <visual>

Commit message: Delete table_link
As panda_arm urdf is used to construct the dual arm urdf, delete the table link. The table link is directly added in the dual arm urdf

File: franka_description/robots/panda_arm.xacro (robot description, xacro)
@@ -11,5 +11,5 @@
       </joint>
     </xacro:unless>
-    <link name="table_link">
+    <!--link name="table_link">
     <visual>
       <geometry>
@@ -23,5 +23,5 @@
       <child link="${arm_id}_link0"/>
       <origin xyz="-0.558 0.175 0.768"/>
-    </joint>
+    </joint-->
     <link name="${arm_id}_link0">
       <visual>
